Commit message: fast funktionierendes python script zum steuern der station

File: src/robot_station/urdf/robot_station.urdf (robot description, URDF)
Before this commit: robot robot_station, 19 links, 18 joints
Joints:
- joint fanuc_joint_1: limit lower=-3.14 upper=3.14 effort=30 velocity=5 -> lower=-3.14 upper=3.14 effort=3000 velocity=5
- joint fanuc_joint_2: limit lower=-3.14 upper=3.14 effort=30 velocity=5 -> lower=-3.14 upper=3.14 effort=3000 velocity=5
- joint fanuc_joint_3: limit lower=-3.14 upper=3.14 effort=30 velocity=5 -> lower=-3.14 upper=3.14 effort=3000 velocity=5
- joint fanuc_joint_4: limit lower=-3.14 upper=3.14 effort=30 velocity=5 -> lower=-3.14 upper=3.14 effort=3000 velocity=5
- joint fanuc_joint_5: limit lower=-3.14 upper=3.14 effort=30 velocity=5 -> lower=-3.14 upper=3.14 effort=300 velocity=5
- joint igus_joint_1: limit lower=0 upper=1.58 effort=30 velocity=5 -> lower=0 upper=1.58 effort=3000 velocity=5
- joint igus_joint_2: limit lower=0 upper=0.47 effort=30 velocity=5 -> lower=0 upper=0.47 effort=3000 velocity=5
- joint igus_joint_3: limit lower=-2.6 upper=2.6 effort=30 velocity=5 -> lower=-2.6 upper=2.6 effort=3000 velocity=5
- joint igus_joint_4: limit lower=-2.6 upper=2.6 effort=30 velocity=5 -> lower=-2.6 upper=2.6 effort=3000 velocity=5
- joint igus_joint_5: limit lower=-2.6 upper=2.6 effort=30 velocity=5 -> lower=-2.6 upper=2.6 effort=3000 velocity=5
- joint rim_joint_1: limit lower=0 upper=3.5 effort=30 velocity=5 -> lower=0 upper=3.5 effort=3000 velocity=5
- joint rim_joint_2: limit lower=0 upper=3.5 effort=30 velocity=5 -> lower=0 upper=3.5 effort=3000 velocity=5
- joint rim_joint_3: limit lower=0 upper=3.5 effort=30 velocity=5 -> lower=0 upper=3.6 effort=3000 velocity=5
